File: KiCAD/AERIS-F411-PCB/POWER.kicad_sch (KiCad schematic)
At the start: 26 parts, among them J1 USB_C_Receptacle_USB2.0_16P, J2 XT30PW-M, Q1 Q_PMOS_GSD, U1 TPS563201DDCR, U2 USBLC6-2SC6, U4 INA219AIDCNR, U9 AMS1117-3.3

Commit message: solve issue of power sheet
Connections:
- net FB: no longer names the net of R2.2, R3.1, U1.4 (VFB)
Changed lines of the file:
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@@
+	(wire
+		(pts
+			(xy 134.62 139.7) (xy 127 139.7)
+		)
+		(stroke
+			(width 0)
+			(type default)
+		)
+	)
 	(wire
 		(pts
@@
 	(wire
 		(pts
-			(xy 228.6 96.52) (xy 237.49 96.52)
+			(xy 228.6 96.52) (xy 251.46 96.52)
 		)
 		(stroke
@@
 	(wire
 		(pts
+			(xy 134.62 157.48) (xy 134.62 139.7)
+		)
+		(stroke
+			(width 0)
+			(type default)
+		)
+	)
+	(wire
+		(pts
 			(xy 228.6 95.25) (xy 228.6 96.52)
 		)
@@
 	(wire
 		(pts
+			(xy 251.46 157.48) (xy 134.62 157.48)
+		)
+		(stroke
+			(width 0)
+			(type default)
+		)
+	)
+	(wire
+		(pts
 			(xy 134.62 41.91) (xy 134.62 43.18)
 		)
@@
 	(wire
 		(pts
+			(xy 127 138.43) (xy 121.92 138.43)
+		)
+		(stroke
+			(width 0)
+			(type default)
+		)
+	)
+	(wire
+		(pts
 			(xy 115.57 113.03) (xy 115.57 109.22)
 		)
@@
 	(wire
 		(pts
+			(xy 127 139.7) (xy 127 138.43)
+		)
+		(stroke
+			(width 0)
+			(type default)
+		)
+	)
+	(wire
+		(pts
+			(xy 212.09 71.12) (xy 214.63 71.12)
+		)
+		(stroke
+			(width 0)
+			(type default)
+		)
+	)
+	(wire
+		(pts
 			(xy 76.2 96.52) (xy 76.2 82.55)
 		)
@@
 	(wire
 		(pts
+			(xy 251.46 96.52) (xy 251.46 157.48)
+		)
+		(stroke
+			(width 0)
+			(type default)
+		)
+	)
+	(wire
+		(pts
 			(xy 129.54 135.89) (xy 134.62 135.89)
 		)
@@
 			(width 0)
 			(type default)
-		)
-	)
-	(label "FB"
-		(at 121.92 138.43 0)
-		(effects
-			(font
-				(size 1.27 1.27)
-			)
-			(justify left bottom)
-		)
-	)
-	(label "U10_VCC"
-		(at 212.09 71.12 0)
-		(effects
-			(font
-				(size 1.27 1.27)
-			)
-			(justify left bottom)
-		)
-	)
-	(label "FB"
-		(at 237.49 96.52 0)
-		(effects
-			(font
-				(size 1.27 1.27)
-			)
-			(justify left bottom)
 		)
 	)
@@
 		)
 	)
+	(hierarchical_label "U10_VCC"
+		(shape output)
+		(at 214.63 71.12 0)
+		(effects
+			(font
+				(size 1.27 1.27)
+			)
+			(justify left)
+		)
+	)
