File: KiCAD/AERIS-F411-PCB/POWER.kicad_sch (KiCad schematic)
At the start: 26 parts, among them J1 USB_C_Receptacle_USB2.0_16P, J2 XT30PW-M, Q1 Q_PMOS_GSD, U1 TPS563201DDCR, U2 USBLC6-2SC6, U4 INA219AIDCNR, U9 AMS1117-3.3

Commit message: Update_in_Power_Section
Parts:
- removed U4: INA219AIDCNR, INA219AIDCNR:SOT65P280X145-8N, symbol INA219AIDCNR:INA219AIDCNR
- removed U9: AMS1117-3.3, Package_TO_SOT_SMD:SOT-223-3_TabPin2, symbol Regulator_Linear:AMS1117-3.3
- added C5c1, C5d1: 1uF, Capacitor_SMD:C_0805_2012Metric, symbol Device:C
- added U10: INA226, Package_SO:TSSOP-10_3x3mm_P0.5mm, symbol Sensor_Energy:INA226
- added U9a1: AP2112K-3.3, Package_TO_SOT_SMD:SOT-23-5, symbol Regulator_Linear:AP2112K-3.3
- added U9b1: AP2112K-3.3, symbol Regulator_Linear:AP2112K-3.3
- C5a1: renamed from C5; value 10uF -> 1uF
- C5b1: renamed from C6; value 22uF -> 1uF
- R2: value 20K -> 51K
- R3: value 6.8K -> 10K
- renumbered J2 to J1, J1 to J2
Connections:
- net +3.3V: now also U9a1.5 (VOUT)
- net +5V: now also C5c1.1, U9a1.1 (VIN), U9a1.3 (EN), U9b1.1 (VIN), U9b1.3 (EN)
- net GND: now also C5c1.2, C5d1.2, U10.1 (A1), U10.2 (A0), U10.7 (GND), U9a1.2 (GND), U9b1.2 (GND)
- net I2C1_SCL: now also U10.5 (SCL)
- net I2C1_SDA: now also U10.4 (SDA)
- net at C1.1, C2.2, R26.2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: now also U10.8 (Vbus), U10.9 (Vin-)
- net +BATT: now reaches J1.P, Q1.3 (D)
- net at D1.1 (A1), F1.2, R26.1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: now also U10.10 (Vin+)
- net USB_DM renamed USB_FS_DM
- net USB_DP renamed USB_FS_DP
- new net +3.3V_SENSOR: C5d1.1, U10.6 (VS), U9b1.5 (VOUT)
- no-connect marks 2 -> 3
Other:
- moved on the sheet: C1, C2, C5a1, C5b1, C7, D1, R26

Commit message: updated
Parts:
- removed D1: D_TVS, Diode_SMD:D_SMB, symbol Device:D_TVS
- removed D2: D_Schottky, Diode_SMD:D_SOD-123, symbol Device:D_Schottky
- added D1: SMBJ12A, SMBJ12A:DIOM4336X265N, symbol SMBJ12A:SMBJ12A
- added D2: B0530W, B0530W:DIO_B0530W, symbol B0530W:B0530W
- C7: value 10nF -> 100nF
- R2: value 51K -> 56K
- R26: value R_Shunt -> 20mohm
- renumbered U9a1 to U9A1, U9b1 to U9B1
Connections:
- net +5V: now also D2.C
- net GND: now also D1.C
- net at J2.A4 (VBUS), J2.A9 (VBUS), J2.B4 (VBUS)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: now also D2.A
- net at F1.2, R26.1, R26.3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: now also D1.A
- net +BATT: no longer names the net of J1.P, Q1.3 (D)

Commit message: update
Changed lines of the file:
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@@
 	)
 	(junction
+		(at 76.2 106.68)
+		(diameter 0)
+		(color 0 0 0 0)
+	)
+	(junction
 		(at 78.74 82.55)
 		(diameter 0)
@@
 	(wire
 		(pts
-			(xy 76.2 99.06) (xy 76.2 111.76)
+			(xy 76.2 99.06) (xy 76.2 106.68)
 		)
 		(stroke
@@
 	(wire
 		(pts
+			(xy 76.2 106.68) (xy 76.2 111.76)
+		)
+		(stroke
+			(width 0)
+			(type default)
+		)
+	)
+	(wire
+		(pts
 			(xy 227.33 137.16) (xy 231.14 137.16)
 		)
@@
 	(wire
 		(pts
-			(xy 66.04 118.11) (xy 66.04 121.92)
-		)
-		(stroke
-			(width 0)
-			(type default)
-		)
-	)
-	(wire
-		(pts
 			(xy 55.88 163.83) (xy 55.88 167.64)
 		)
@@
 	(wire
 		(pts
-			(xy 66.04 151.13) (xy 66.04 153.67)
-		)
-		(stroke
-			(width 0)
-			(type default)
-		)
-	)
-	(wire
-		(pts
 			(xy 146.05 148.59) (xy 144.78 148.59)
 		)
@@
 	)
 	(symbol
-		(lib_id "power:PWR_FLAG")
-		(at 66.04 118.11 0)
-		(unit 1)
-		(body_style 1)
-		(exclude_from_sim no)
-		(in_bom yes)
-		(on_board yes)
-		(in_pos_files yes)
-		(dnp no)
-		(fields_autoplaced yes)
-		(property "Reference" "#FLG02"
-			(at 66.04 116.205 0)
-			(hide yes)
-			(show_name no)
-			(do_not_autoplace no)
-			(effects
-				(font
-					(size 1.27 1.27)
-				)
-			)
-		)
-		(property "Value" "PWR_FLAG"
-			(at 66.04 113.03 0)
-			(show_name no)
-			(do_not_autoplace no)
-			(effects
-				(font
-					(size 1.27 1.27)
-				)
-			)
-		)
-		(property "Footprint" ""
-			(at 66.04 118.11 0)
-			(hide yes)
-			(show_name no)
-			(do_not_autoplace no)
-			(effects
-				(font
-					(size 1.27 1.27)
-				)
-			)
-		)
-		(property "Datasheet" ""
-			(at 66.04 118.11 0)
-			(hide yes)
-			(show_name no)
-			(do_not_autoplace no)
-			(effects
-				(font
-					(size 1.27 1.27)
-				)
-			)
-		)
-		(property "Description" "Special symbol for telling ERC where power comes from"
-			(at 66.04 118.11 0)
-			(hide yes)
-			(show_name no)
-			(do_not_autoplace no)
-			(effects
-				(font
-					(size 1.27 1.27)
-				)
-			)
-		)
-		(pin "1"
-		)
-		(instances
-			(project "AERIS-F411-PCB"
-				(path "/41f25c5f-e761-4f33-a9f5-6d8db67ffdd9/0e6091cd-36a8-495e-bc03-729bcaf76ce2"
-					(reference "#FLG02")
-					(unit 1)
-				)
-			)
-		)
-	)
-	(symbol
 		(lib_id "Regulator_Linear:AP2112K-3.3")
 		(at 55.88 156.21 0)
@@
 	)
 	(symbol
+		(lib_id "power:PWR_FLAG")
+		(at 76.2 106.68 90)
+		(unit 1)
+		(body_style 1)
+		(exclude_from_sim no)
+		(in_bom yes)
+		(on_board yes)
+		(in_pos_files yes)
+		(dnp no)
+		(fields_autoplaced yes)
+		(property "Reference" "#FLG02"
+			(at 74.295 106.68 0)
+			(hide yes)
+			(show_name no)
+			(do_not_autoplace no)
+			(effects
+				(font
+					(size 1.27 1.27)
+				)
+			)
+		)
+		(property "Value" "PWR_FLAG"
+			(at 72.39 106.6799 90)
+			(show_name no)
+			(do_not_autoplace no)
+			(effects
+				(font
+					(size 1.27 1.27)
+				)
+				(justify left)
+			)
+		)
+		(property "Footprint" ""
+			(at 76.2 106.68 0)
+			(hide yes)
+			(show_name no)
+			(do_not_autoplace no)
+			(effects
+				(font
+					(size 1.27 1.27)
+				)
+			)
+		)
+		(property "Datasheet" ""
+			(at 76.2 106.68 0)
+			(hide yes)
+			(show_name no)
+			(do_not_autoplace no)
+			(effects
+				(font
+					(size 1.27 1.27)
+				)
+			)
+		)
+		(property "Description" "Special symbol for telling ERC where power comes from"
+			(at 76.2 106.68 0)
+			(hide yes)
+			(show_name no)
+			(do_not_autoplace no)
+			(effects
+				(font
+					(size 1.27 1.27)
+				)
+			)
+		)
+		(pin "1"
+		)
+		(instances
+			(project "AERIS-F411-PCB"
+				(path "/41f25c5f-e761-4f33-a9f5-6d8db67ffdd9/0e6091cd-36a8-495e-bc03-729bcaf76ce2"
+					(reference "#FLG02")
+					(unit 1)
+				)
+			)
+		)
+	)
+	(symbol
 		(lib_id "Device:Fuse")
 		(at 95.25 97.79 90)
@@
 					(unit 1)
 				)
-			)
-		)
-	)
-	(symbol
-		(lib_id "power:PWR_FLAG")
-		(at 66.04 151.13 0)
-		(unit 1)
-		(body_style 1)
-		(exclude_from_sim no)
-		(in_bom yes)
-		(on_board yes)
-		(in_pos_files yes)
-		(dnp no)
-		(fields_autoplaced yes)
-		(property "Reference" "#FLG04"
-			(at 66.04 149.225 0)
-			(hide yes)
-			(show_name no)
-			(do_not_autoplace no)
-			(effects
-				(font
-					(size 1.27 1.27)
-				)
-			)
-		)
-		(property "Value" "PWR_FLAG"
-			(at 66.04 146.05 0)
-			(show_name no)
-			(do_not_autoplace no)
-			(effects
-				(font
-					(size 1.27 1.27)
-				)
-			)
-		)
-		(property "Footprint" ""
-			(at 66.04 151.13 0)
-			(hide yes)
-			(show_name no)
-			(do_not_autoplace no)
-			(effects
-				(font
-					(size 1.27 1.27)
-				)
-			)
-		)
-		(property "Datasheet" ""
-			(at 66.04 151.13 0)
-			(hide yes)
-			(show_name no)
-			(do_not_autoplace no)
-			(effects
-				(font
-					(size 1.27 1.27)
-				)
-			)
-		)
-		(property "Description" "Special symbol for telling ERC where power comes from"
-			(at 66.04 151.13 0)
-			(hide yes)
-			(show_name no)
-			(do_not_autoplace no)
-			(effects
-				(font
-					(size 1.27 1.27)
-				)
-			)
-		)
-		(pin "1"
-		)
-		(instances
-			(project "AERIS-F411-PCB"
-				(path "/41f25c5f-e761-4f33-a9f5-6d8db67ffdd9/0e6091cd-36a8-495e-bc03-729bcaf76ce2"
-					(reference "#FLG04")
-					(unit 1)
-				)

Commit message: Update
Parts:
- U9B1: footprint (none) -> Footprints:SOT95P285X145-5N
Connections:
- net GND: now also J2.A7 (D-), J2.B7 (D-), R4.1, U2.2, U2.5
Other:
- moved on the sheet: R4
Changed lines of the file:
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@@
 	)
 	(junction
+		(at 232.41 137.16)
+		(diameter 0)
+		(color 0 0 0 0)
+	)
+	(junction
 		(at 106.68 97.79)
 		(diameter 0)
@@
 	)
 	(junction
+		(at 184.15 137.16)
+		(diameter 0)
+		(color 0 0 0 0)
+	)
+	(junction
 		(at 134.62 92.71)
 		(diameter 0)
@@
 	)
 	(junction
+		(at 184.15 149.86)
+		(diameter 0)
+		(color 0 0 0 0)
+	)
+	(junction
+		(at 232.41 149.86)
+		(diameter 0)
+		(color 0 0 0 0)
+	)
+	(junction
 		(at 55.88 167.64)
 		(diameter 0)
@@
 	(wire
 		(pts
+			(xy 184.15 149.86) (xy 186.69 149.86)
+		)
+		(stroke
+			(width 0)
+			(type default)
+		)
+	)
+	(wire
+		(pts
 			(xy 45.72 167.64) (xy 55.88 167.64)
 		)
@@
 	(wire
 		(pts
-			(xy 227.33 137.16) (xy 231.14 137.16)
+			(xy 227.33 137.16) (xy 232.41 137.16)
 		)
 		(stroke
@@
 	(wire
 		(pts
+			(xy 184.15 137.16) (xy 184.15 149.86)
+		)
+		(stroke
+			(width 0)
+			(type default)
+		)
+	)
+	(wire
+		(pts
 			(xy 163.83 45.72) (xy 167.64 45.72)
 		)
@@
 	(wire
 		(pts
+			(xy 181.61 149.86) (xy 184.15 149.86)
+		)
+		(stroke
+			(width 0)
+			(type default)
+		)
+	)
+	(wire
+		(pts
 			(xy 45.72 166.37) (xy 45.72 167.64)
 		)
@@
 	(wire
 		(pts
+			(xy 232.41 137.16) (xy 234.95 137.16)
+		)
+		(stroke
+			(width 0)
+			(type default)
+		)
+	)
+	(wire
+		(pts
 			(xy 86.36 128.27) (xy 86.36 113.03)
 		)
@@
 	(wire
 		(pts
-			(xy 186.69 137.16) (xy 179.07 137.16)
+			(xy 186.69 137.16) (xy 184.15 137.16)
 		)
 		(stroke
@@
 	(wire
 		(pts
+			(xy 232.41 137.16) (xy 232.41 149.86)
+		)
+		(stroke
+			(width 0)
+			(type default)
+		)
+	)
+	(wire
+		(pts
 			(xy 144.78 148.59) (xy 143.51 148.59)
 		)
@@
 	(wire
 		(pts
+			(xy 245.11 137.16) (xy 242.57 137.16)
+		)
+		(stroke
+			(width 0)
+			(type default)
+		)
+	)
+	(wire
+		(pts
 			(xy 125.73 100.33) (xy 125.73 101.6)
 		)
@@
 	(wire
 		(pts
+			(xy 234.95 149.86) (xy 232.41 149.86)
+		)
+		(stroke
+			(width 0)
+			(type default)
+		)
+	)
+	(wire
+		(pts
+			(xy 184.15 137.16) (xy 179.07 137.16)
+		)
+		(stroke
+			(width 0)
+			(type default)
+		)
+	)
+	(wire
+		(pts
+			(xy 232.41 149.86) (xy 227.33 149.86)
+		)
+		(stroke
+			(width 0)
+			(type default)
+		)
+	)
+	(wire
+		(pts
 			(xy 125.73 101.6) (xy 127 101.6)
 		)
@@
 	(hierarchical_label "USB_FS_DM"
 		(shape bidirectional)
-		(at 238.76 137.16 0)
+		(at 245.11 137.16 0)
 		(effects
 			(font
@@
 			)
 		)
-		(property "Footprint" ""
+		(property "Footprint" "Footprints:SOT95P285X145-5N"
 			(at 55.88 147.955 0)
 			(hide yes)
@@
 	(symbol
 		(lib_id "Device:R")
-		(at 234.95 137.16 90)
+		(at 238.76 137.16 90)
 		(unit 1)
 		(body_style 1)
@@
 		(fields_autoplaced yes)
 		(property "Reference" "R4"
-			(at 234.95 130.81 90)
+			(at 238.76 130.81 90)
 			(show_name no)
 			(do_not_autoplace no)
@@
 		)
 		(property "Value" "22"
-			(at 234.95 133.35 90)
+			(at 238.76 133.35 90)
 			(show_name no)
 			(do_not_autoplace no)
@@
 		)
 		(property "Footprint" "Resistor_SMD:R_0603_1608Metric"
-			(at 234.95 138.938 90)
+			(at 238.76 138.938 90)
 			(hide yes)
 			(show_name no)
@@
 		)
 		(property "Datasheet" ""
-			(at 234.95 137.16 0)
+			(at 238.76 137.16 0)
 			(hide yes)
 			(show_name no)
@@
 		)
 		(property "Description" "Resistor"
-			(at 234.95 137.16 0)
+			(at 238.76 137.16 0)
 			(hide yes)
 			(show_name no)
@@
 		)
 		(property "Purpose" ""
-			(at 234.95 137.16 0)
+			(at 238.76 137.16 0)
 			(show_name no)
 			(do_not_autoplace no)
@@
 	(symbol
 		(lib_id "power:GND")
-		(at 186.69 149.86 270)
+		(at 181.61 149.86 270)
 		(unit 1)
 		(body_style 1)
@@
 		(fields_autoplaced yes)
 		(property "Reference" "#PWR011"
-			(at 180.34 149.86 0)
+			(at 175.26 149.86 0)
 			(hide yes)
 			(show_name no)
@@
 		)
 		(property "Value" "GND"
-			(at 182.88 149.8599 90)
+			(at 177.8 149.8599 90)
 			(show_name no)
 			(do_not_autoplace no)
@@
 		)
 		(property "Footprint" ""
-			(at 186.69 149.86 0)
+			(at 181.61 149.86 0)
 			(hide yes)
 			(show_name no)
@@
 		)
 		(property "Datasheet" ""
-			(at 186.69 149.86 0)
+			(at 181.61 149.86 0)
 			(hide yes)
 			(show_name no)
@@
 		)
 		(property "Description" "Power symbol creates a global label with name \"GND\" , ground"
-			(at 186.69 149.86 0)
+			(at 181.61 149.86 0)
 			(hide yes)
 			(show_name no)
@@
 	(symbol
 		(lib_id "power:GND")
-		(at 227.33 149.86 90)
+		(at 234.95 149.86 90)
 		(unit 1)
 		(body_style 1)
@@
 		(fields_autoplaced yes)
 		(property "Reference" "#PWR010"
-			(at 233.68 149.86 0)
+			(at 241.3 149.86 0)
 			(hide yes)
 			(show_name no)
@@
 		)
 		(property "Value" "GND"
-			(at 231.14 149.8599 90)
+			(at 238.76 149.8599 90)
 			(show_name no)
 			(do_not_autoplace no)
@@
 		)
 		(property "Footprint" ""
-			(at 227.33 149.86 0)
+			(at 234.95 149.86 0)
 			(hide yes)
 			(show_name no)
@@
 		)
 		(property "Datasheet" ""
-			(at 227.33 149.86 0)
+			(at 234.95 149.86 0)
 			(hide yes)
 			(show_name no)
@@
 		)
 		(property "Description" "Power symbol creates a global label with name \"GND\" , ground"
-			(at 227.33 149.86 0)
+			(at 234.95 149.86 0)
 			(hide yes)
 			(show_name no)
