File: KiCAD/AERIS-F411-PCB/MCU_Core.kicad_sch (KiCad schematic)
At the start: 0 parts

Commit message: Update
Parts:
- added C10, C16, C18, C21, C22, C23, C24, C5, C8: 100nF, Capacitor_SMD:C_0603_1608Metric, symbol Device:C
- added C11, C14: 3.9pF, Capacitor_SMD:C_0603_1608Metric, symbol Device:C
- added C12, C15: 2.2uF, Capacitor_SMD:C_0603_1608Metric, symbol Device:C
- added C13, C6: 1uF, Capacitor_SMD:C_0603_1608Metric, symbol Device:C
- added C17, C20: 1.5pF, Capacitor_SMD:C_0603_1608Metric, symbol Device:C
- added C19: 4.7uF, Capacitor_SMD:C_0603_1608Metric, symbol Device:C
- added C9: 4.7uF, Capacitor_SMD:C_0805_2012Metric, symbol Device:C
- added FB1: FerriteBead_Small, Inductor_SMD:L_0603_1608Metric, symbol Device:FerriteBead_Small
- added J3: Conn_01x06, Connector_PinHeader_1.00mm:PinHeader_2x03_P1.00mm_Vertical, symbol Connector_Generic:Conn_01x06
- added R8: 10kohm, Resistor_SMD:R_0603_1608Metric, symbol Device:R
- added R9: 0, Resistor_SMD:R_0603_1608Metric, symbol Device:R
- added SW1, SW2: SW_Push, Button_Switch_SMD:SW_SPST_B3U-1000P, symbol Switch:SW_Push
- added U3: STM32H743VITx, Package_QFP:LQFP-100_14x14mm_P0.5mm, symbol MCU_ST_STM32H7:STM32H743VITx
- added Y1: 25 MHz, Crystal:Crystal_SMD_3225-4Pin_3.2x2.5mm, symbol Device:Crystal_GND24
- added Y2: 32.768kHz, Crystal:Crystal_SMD_3215-2Pin_3.2x1.5mm, symbol Device:Crystal_GND24_Small
Connections:
- new net: Y2.2 (G), Y2.4 (G)
- new net: C12.1, U3.48 (VCAP)
- new net: R9.1, U3.20 (VREF+)
- new net: C18.1, C6.2, FB1.1, R9.2, U3.21 (VDDA)
- new net: C18.2, C6.1, U3.19 (VSSA)
- new net: C15.1, U3.73 (VCAP)
- new net: Y1.2 (G), Y1.4 (G)
- new net 3.3V: C21.1, C22.1, C23.1, C24.1, C5.1, C9.1, FB1.2, U3.100 (VDD), U3.11 (VDD), U3.27 (VDD), U3.50 (VDD), U3.75 (VDD)
- new net GND: C21.2, C22.2, C23.2, C24.2, C5.2, C9.2, U3.10 (VSS), U3.26 (VSS), U3.49 (VSS), U3.74 (VSS), U3.99 (VSS)

Commit message: MCU Core ADDED
Parts:
- removed C19: 4.7uF, Capacitor_SMD:C_0603_1608Metric, symbol Device:C
Connections:
- net 3.3V: now also J3.1 (Pin_1), SW2.2
- net GND: now also C11.2, C12.2, C14.2, C15.2, C16.2, C17.2, C20.2, C8.2, J3.3 (Pin_3), R8.2, SW1.2, Y1.2 (G), Y1.4 (G), Y2.2 (G), Y2.4 (G)
- net PC14: now reaches Y2.1
- net PC14: now also C17.1, U3.8 (PC14)
- net PC15: now reaches Y2.3
- net PC15: now also C20.1, U3.9 (PC15)
- net NRST: now reaches C8.1
- net NRST: now also J3.5 (Pin_5), SW1.1, U3.14 (NRST)
- net VREF: now reaches C13.1
- net VREF: now also C10.1, R9.1, U3.20 (VREF+)
- net VSSA: now reaches C13.2
- net VSSA: now also C10.2, C18.2, C6.1, U3.19 (VSSA)
- net at R8.1: now also SW2.1, U3.94 (BOOT0)
- net PH0: now reaches U3.12 (PH0)
- net PH0: now also C11.1, Y1.1
- net PH1: now reaches U3.13 (PH1)
- net PH1: now also C14.1, Y1.3
- net at U3.6 (VBAT): now also C16.1
- net at U3.72 (PA13): now also J3.2 (Pin_2)
- net at U3.76 (PA14): now also J3.4 (Pin_4)
- net at U3.89 (PB3): now also J3.6 (Pin_6)
- no-connect marks 0 -> 75
Other:
- moved on the sheet: C10, C11, C13, C14, C16, C17, C20, C23, C8, J3, R8, R9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

Commit message: Added Memory/Storage sheet
Connections:
- net 3.3V renamed +3.3V
Changed lines of the file:
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@@
 		)
 	)
-	(hierarchical_label "3.3V"
+	(hierarchical_label "+3.3V"
 		(shape input)
 		(at 124.46 138.43 0)
@@
 		)
 	)
-	(hierarchical_label "3.3V"
+	(hierarchical_label "+3.3V"
 		(shape input)
 		(at 250.19 35.56 180)
@@
 		)
 	)
-	(hierarchical_label "3.3V"
+	(hierarchical_label "+3.3V"
 		(shape input)
 		(at 58.42 90.17 180)
