File: KiCAD/AERIS-F411-PCB/AERIS-F411-PCB.kicad_pcb (KiCad board)
At the start: 2 copper layers, 22 parts, among them J1 USB_C_Receptacle_USB2.0_16P, Q1 Q_PMOS_GSD, U9 AMS1117-3.3

Commit message: update
Parts:
- added C10: 100nF, Capacitor_SMD:C_0603_1608Metric, F.Cu at (164.1, 87.1)
- added C11: 3.9pF, Capacitor_SMD:C_0603_1608Metric, F.Cu at (164.1, 89.6)
- added C12: 2.2uF, Capacitor_SMD:C_0603_1608Metric, F.Cu at (168.1, 79.6)
- added C13: 1uF, Capacitor_SMD:C_0603_1608Metric, F.Cu at (168.1, 82.1)
- added C14: 3.9pF, Capacitor_SMD:C_0603_1608Metric, F.Cu at (168.1, 84.6)
- added C15: 2.2uF, Capacitor_SMD:C_0603_1608Metric, F.Cu at (168.1, 87.1)
- added C16: 100nF, Capacitor_SMD:C_0603_1608Metric, F.Cu at (168.1, 89.6)
- added C17: 1.5pF, Capacitor_SMD:C_0603_1608Metric, F.Cu at (172.1, 79.6)
- added C18: 100nF, Capacitor_SMD:C_0603_1608Metric, F.Cu at (172.1, 82.1)
- added C20: 1.5pF, Capacitor_SMD:C_0603_1608Metric, F.Cu at (172.1, 84.6)
- added C21: 100nF, Capacitor_SMD:C_0603_1608Metric, F.Cu at (172.1, 87.1)
- added C22: 100nF, Capacitor_SMD:C_0603_1608Metric, F.Cu at (172.1, 89.6)
- added C23: 100nF, Capacitor_SMD:C_0603_1608Metric, F.Cu at (176.1, 79.6)
- added C24: 100nF, Capacitor_SMD:C_0603_1608Metric, F.Cu at (176.1, 82.1)
- added C25: 100nF, Capacitor_SMD:C_0603_1608Metric, F.Cu at (201.5, 63.0)
- added C26: 1uF, Capacitor_SMD:C_0603_1608Metric, F.Cu at (201.5, 65.5)
- added C5: 100nF, Capacitor_SMD:C_0603_1608Metric, F.Cu at (164.1, 79.6)
- added C5c1: 1uF, Capacitor_SMD:C_0805_2012Metric, F.Cu at (190.0, 65.9)
- added C5d1: 1uF, Capacitor_SMD:C_0805_2012Metric, F.Cu at (190.0, 68.9)
- added C6: 1uF, Capacitor_SMD:C_0603_1608Metric, F.Cu at (164.1, 82.1)
- added C8: 100nF, Capacitor_SMD:C_0603_1608Metric, F.Cu at (164.1, 84.6)
- added C9: 4.7uF, Capacitor_SMD:C_0805_2012Metric, F.Cu at (182.8, 74.3)
- added FB1: FerriteBead_Small, Inductor_SMD:L_0603_1608Metric, F.Cu at (176.1, 84.6)
- added J3: Conn_01x06, Connector_PinHeader_1.00mm:PinHeader_2x03_P1.00mm_Vertical, F.Cu at (182.2, 69.2)
- added R10: 10k, Resistor_SMD:R_0603_1608Metric, F.Cu at (201.5, 68.0)
- added R11: 10k, Resistor_SMD:R_0603_1608Metric, F.Cu at (201.5, 70.6)
- added R12: 47k, Resistor_SMD:R_0603_1608Metric, F.Cu at (201.5, 73.1)
- added R13: 47k, Resistor_SMD:R_0603_1608Metric, F.Cu at (201.5, 75.6)
- added R14: 47k, Resistor_SMD:R_0603_1608Metric, F.Cu at (201.5, 78.1)
- added R15: 47k, Resistor_SMD:R_0603_1608Metric, F.Cu at (201.5, 80.6)
- added R16: 47k, Resistor_SMD:R_0603_1608Metric, F.Cu at (201.5, 83.1)
- added R8: 10kohm, Resistor_SMD:R_0603_1608Metric, F.Cu at (176.1, 87.1)
- added R9: 0, Resistor_SMD:R_0603_1608Metric, F.Cu at (176.1, 89.6)
- added SW1: SW_Push, Button_Switch_SMD:SW_SPST_B3U-1000P, F.Cu at (181.0, 80.5)
- added SW2: SW_Push, Button_Switch_SMD:SW_SPST_B3U-1000P, F.Cu at (181.0, 84.9)
- added U10: INA226, Package_SO:TSSOP-10_3x3mm_P0.5mm, F.Cu at (191.5, 62.1)
- added U3: STM32H743VITx, Package_QFP:LQFP-100_14x14mm_P0.5mm, F.Cu at (171.3, 69.1)
- added U5: W25Q128JVS, Package_SO:SOIC-8_5.3x5.3mm_P1.27mm, F.Cu at (193.0, 79.2)
- added U9A1: AP2112K-3.3, Package_TO_SOT_SMD:SOT-23-5, F.Cu at (194.8, 71.4)
- added U9B1: AP2112K-3.3, Footprints:SOT95P285X145-5N, F.Cu at (195.1, 66.7)
- added Y1: 25 MHz, Crystal:Crystal_SMD_3225-4Pin_3.2x2.5mm, F.Cu at (183.2, 62.1)
- added Y2: 32.768kHz, Crystal:Crystal_SMD_3215-2Pin_3.2x1.5mm, F.Cu at (183.1, 66.0)
- C5a1: renamed from C5; value 10uF -> 1uF
- C5b1: renamed from C6; value 22uF -> 1uF
- C7: value 10nF -> 100nF
- R2: value 20K -> 56K
- R26: value R_Shunt -> 20mohm
- R3: value 6.8K -> 10K
- renumbered J1 to J2
Connections:
- net /POWER SECTION/FB renamed Net-(U1-VFB)
- net /POWER SECTION/USB_DM renamed /POWER SECTION/USB_FS_DM
- net /POWER SECTION/USB_DP renamed /POWER SECTION/USB_FS_DP
- C1 pad 2: /POWER SECTION/GND -> GND
- C2 pad 1: /POWER SECTION/GND -> GND
- C3 pad 1: /POWER SECTION/GND -> GND
- C3 pad 2: /POWER SECTION/5V -> /POWER SECTION/+5V
- C5a1 pad 1: /POWER SECTION/5V -> /POWER SECTION/+5V
- C5a1 pad 2: /POWER SECTION/GND -> GND
- C5b1 pad 1: /POWER SECTION/3.3V -> /MCU_Core/+3.3V
- C5b1 pad 2: /POWER SECTION/GND -> GND
- C7 pad 2: /POWER SECTION/GND -> GND
- F1 pad 2: Net-(D1-A1) -> Net-(U10-Vin+)
- J2 pad A1: /POWER SECTION/GND -> GND
- J2 pad A12: /POWER SECTION/GND -> GND
- J2 pad A4: Net-(D2-A) -> Net-(D2-PadA)
- J2 pad A7: Net-(J1-D--PadA7) -> GND
- J2 pad A9: Net-(D2-A) -> Net-(D2-PadA)
- J2 pad B1: /POWER SECTION/GND -> GND
- J2 pad B12: /POWER SECTION/GND -> GND
- J2 pad B4: Net-(D2-A) -> Net-(D2-PadA)
- J2 pad B7: Net-(J1-D--PadA7) -> GND
- J2 pad B9: Net-(D2-A) -> Net-(D2-PadA)
- J2 pad SH: /POWER SECTION/GND -> GND
- L1 pad 1: /POWER SECTION/5V -> /POWER SECTION/+5V
- R1 pad 2: /POWER SECTION/GND -> GND
- R2 pad 1: /POWER SECTION/5V -> /POWER SECTION/+5V
- R26 pad 1: Net-(D1-A1) -> Net-(U10-Vin+)
- R3 pad 2: /POWER SECTION/GND -> GND
- R4 pad 1: Net-(R4-Pad1) -> GND
- R6 pad 1: /POWER SECTION/GND -> GND
- R7 pad 2: /POWER SECTION/GND -> GND
