File: KiCAD/AERIS-H743-PCB/Conn&Inc.kicad_sch (KiCad schematic)
At the start: 19 parts, among them J10 ESC1, J11 ESC2, J12 ESC3, J13 ESC4, SW3 SW_Push

Commit message: Updated and complete Schematic
Parts:
- removed D3: LED3, LED_SMD:LED_0603_1608Metric, symbol Device:LED
- added D6: LED_RGB, LED_SMD:LED_RGB_5050-6, symbol Device:LED_RGB
Connections:
- net GND: now also C33.2, D4.1 (K), D5.1 (K), SW3.2, D6.1 (RK), D6.2 (GK), D6.3 (BK)
- net RGB_G: now reaches R32.1
- net at R32.2: now also D6.5 (GA)
- net +3V3: now reaches R31.1
- net +3V3: now also R22.1
- net USER_BTN: now reaches R31.2
- net USER_BTN: now also C33.1, SW3.1
- net at D5.2 (A): now also R22.2
- net at R28.1: now also D6.6 (RA)
- net RGB_R: now reaches R28.2
- net at R25.1: now also D4.2 (A)
- net Status_LED: now reaches R25.2
- net at R30.1: now also D6.4 (BA)
- net RGB_B: now reaches R30.2
- no-connect marks 0 -> 4
Other:
- moved on the sheet: D4, D5, J10, J11, J12, J13, R22, R23, R24, R25, R27, R28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
