File: KiCAD/AERIS-H743-PCB/Memory&Storage.kicad_sch (KiCad schematic)
At the start: 12 parts, among them J4 1040310811, U5 W25Q128JVS

Commit message: Sensor Sheet Updated
Parts:
- C19: footprint (none) -> Capacitor_SMD:C_0603_1608Metric
Changed lines of the file:
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@@
 		)
 		(instances
-			(project "AERIS-F411-PCB"
+			(project "AERIS-H743-PCB"
 				(path "/41f25c5f-e761-4f33-a9f5-6d8db67ffdd9/f01385d2-11fb-4f45-b9f3-8008279d6804"
 					(reference "#PWR031")
@@
 		)
 		(instances
-			(project "AERIS-F411-PCB"
+			(project "AERIS-H743-PCB"
 				(path "/41f25c5f-e761-4f33-a9f5-6d8db67ffdd9/f01385d2-11fb-4f45-b9f3-8008279d6804"
 					(reference "R15")
@@
 		)
 		(instances
-			(project "AERIS-F411-PCB"
+			(project "AERIS-H743-PCB"
 				(path "/41f25c5f-e761-4f33-a9f5-6d8db67ffdd9/f01385d2-11fb-4f45-b9f3-8008279d6804"
 					(reference "R16")
@@
 		)
 		(instances
-			(project "AERIS-F411-PCB"
+			(project "AERIS-H743-PCB"
 				(path "/41f25c5f-e761-4f33-a9f5-6d8db67ffdd9/f01385d2-11fb-4f45-b9f3-8008279d6804"
 					(reference "#PWR030")
@@
 		)
 		(instances
-			(project "AERIS-F411-PCB"
+			(project "AERIS-H743-PCB"
 				(path "/41f25c5f-e761-4f33-a9f5-6d8db67ffdd9/f01385d2-11fb-4f45-b9f3-8008279d6804"
 					(reference "R11")
@@
 		)
 		(instances
-			(project "AERIS-F411-PCB"
+			(project "AERIS-H743-PCB"
 				(path "/41f25c5f-e761-4f33-a9f5-6d8db67ffdd9/f01385d2-11fb-4f45-b9f3-8008279d6804"
 					(reference "R13")
@@
 		)
 		(instances
-			(project "AERIS-F411-PCB"
+			(project "AERIS-H743-PCB"
 				(path "/41f25c5f-e761-4f33-a9f5-6d8db67ffdd9/f01385d2-11fb-4f45-b9f3-8008279d6804"
 					(reference "R14")
@@
 		)
 		(instances
-			(project "AERIS-F411-PCB"
+			(project "AERIS-H743-PCB"
 				(path "/41f25c5f-e761-4f33-a9f5-6d8db67ffdd9/f01385d2-11fb-4f45-b9f3-8008279d6804"
 					(reference "#PWR029")
@@
 		)
 		(instances
-			(project "AERIS-F411-PCB"
+			(project "AERIS-H743-PCB"
 				(path "/41f25c5f-e761-4f33-a9f5-6d8db67ffdd9/f01385d2-11fb-4f45-b9f3-8008279d6804"
 					(reference "R12")
@@
 		)
 		(instances
-			(project "AERIS-F411-PCB"
+			(project "AERIS-H743-PCB"
 				(path "/41f25c5f-e761-4f33-a9f5-6d8db67ffdd9/f01385d2-11fb-4f45-b9f3-8008279d6804"
 					(reference "C26")
@@
 			)
 		)
-		(property "Footprint" ""
+		(property "Footprint" "Capacitor_SMD:C_0603_1608Metric"
 			(at 69.85 66.3448 0)
 			(hide yes)
@@
 		)
 		(instances
-			(project "AERIS-F411-PCB"
+			(project "AERIS-H743-PCB"
 				(path "/41f25c5f-e761-4f33-a9f5-6d8db67ffdd9/f01385d2-11fb-4f45-b9f3-8008279d6804"
 					(reference "C19")
@@
 		)
 		(instances
-			(project "AERIS-F411-PCB"
+			(project "AERIS-H743-PCB"
 				(path "/41f25c5f-e761-4f33-a9f5-6d8db67ffdd9/f01385d2-11fb-4f45-b9f3-8008279d6804"
 					(reference "C25")
@@
 		)
 		(instances
-			(project "AERIS-F411-PCB"
+			(project "AERIS-H743-PCB"
 				(path "/41f25c5f-e761-4f33-a9f5-6d8db67ffdd9/f01385d2-11fb-4f45-b9f3-8008279d6804"
 					(reference "R10")
@@
 		)
 		(instances
-			(project "AERIS-F411-PCB"
+			(project "AERIS-H743-PCB"
 				(path "/41f25c5f-e761-4f33-a9f5-6d8db67ffdd9/f01385d2-11fb-4f45-b9f3-8008279d6804"
 					(reference "J4")
@@
 		)
 		(instances
-			(project "AERIS-F411-PCB"
+			(project "AERIS-H743-PCB"
 				(path "/41f25c5f-e761-4f33-a9f5-6d8db67ffdd9/f01385d2-11fb-4f45-b9f3-8008279d6804"
 					(reference "U5")

Commit message: Update
Parts:
- removed J4: 1040310811, 1040310811:104031-0811_MOL, symbol 1040310811:1040310811
- added J4: 1040310811, Library:104031-0811_MOL, symbol 104031-0811_MOL:1040310811
Connections:
- net +3V3: now also J4.4 (VDD)
- net GND: now also J4.6 (VSS)
- net SDMMC_CLK: now also J4.5 (CLK)
- net SDMMC_CMD: now also J4.3 (CMD)
- net SDMMC_D0: now also J4.7 (DAT0)
- net SDMMC_D1: now also J4.8 (DAT1)
- net SDMMC_D2: now also J4.1 (DAT2)
- net SDMMC_D3: now also J4.2 (CD/DAT3)
