File: KiCAD/AERIS-H743-PCB/MCU_Core.kicad_sch (KiCad schematic)
At the start: 27 parts, among them J3 Conn_01x06, SW1 SW_Push, SW2 SW_Push, U3 STM32H743VITx, Y1 25 MHz, Y2 32.768kHz

Commit message: Sensor Sheet Updated
Connections:
- net SPI1_NSS: now reaches U3.28 (PA4)
- net SPI1_SCK: now reaches U3.29 (PA5)
- net SPI1_MISO: now reaches U3.30 (PA6)
- net SPI1_MOSI: now reaches U3.31 (PA7)
- net I2C1_SCL: now reaches U3.95 (PB8)
- net I2C1_SDA: now reaches U3.96 (PB9)
- net +3.3V renamed +3V3
- no-connect marks 75 -> 69

Commit message: Updated and complete Schematic
Connections:
- net QSPI_IO2: now reaches U3.1 (PE2)
- net IMU_INT1: now reaches U3.15 (PC0)
- net USER_BTN: now reaches U3.16 (PC1)
- net Status_LED: now reaches U3.17 (PC2_C)
- net RGB_R: now reaches U3.18 (PC3_C)
- net RGB_G: now reaches U3.32 (PC4)
- net RGB_B: now reaches U3.33 (PC5)
- net QSPI_CLK: now reaches U3.36 (PB2)
- net ESC1_PWM: now reaches U3.39 (PE9)
- net ESC2_PWM: now reaches U3.41 (PE11)
- net ESC3_PWM: now reaches U3.43 (PE13)
- net ESC4_PWM: now reaches U3.44 (PE14)
- net RS485_TX: now reaches U3.55 (PD8)
- net RS485_RX: now reaches U3.56 (PD9)
- net RS485_DE: now reaches U3.57 (PD10)
- net QSPI_IO0: now reaches U3.58 (PD11)
- net QSPI_IO1: now reaches U3.59 (PD12)
- net QSPI_IO3: now reaches U3.60 (PD13)
- net SDMMC_D0: now reaches U3.65 (PC8)
- net SDMMC_D1: now reaches U3.66 (PC9)
- net USP_DM: now reaches U3.70 (PA11)
- net USB_DP: now reaches U3.71 (PA12)
- net SDMMC_D2: now reaches U3.78 (PC10)
- net SDMMC_D3: now reaches U3.79 (PC11)
- net SDMMC_CLK: now reaches U3.80 (PC12)
- net FDCAN_RX: now reaches U3.81 (PD0)
- net FDCAN_TX: now reaches U3.82 (PD1)
- net SDMMC_CMD: now reaches U3.83 (PD2)
- net QSPI_NCS: now reaches U3.92 (PB6)
- net GPS_RX: now reaches U3.97 (PE0)
- net GPS_TX: now reaches U3.98 (PE1)
- no-connect marks 69 -> 38

Commit message: Update
Parts:
- removed Y2: 32.768kHz, Crystal:Crystal_SMD_3215-2Pin_3.2x1.5mm, symbol Device:Crystal_GND24_Small
- added Y2: 32.768KHz, Crystal:Crystal_SMD_3215-2Pin_3.2x1.5mm, symbol Device:Crystal
Connections:
- net PC14: now also Y2.1
- net PC15: now also Y2.2
Other:
- moved on the sheet: C17, C20
