File: KiCAD/AERIS-H743-PCB/POWER.kicad_sch (KiCad schematic)
At the start: 29 parts, among them J1 XT30PW-M, J2 USB_C_Receptacle_USB2.0_16P, Q1 Q_PMOS_GSD, U1 TPS563201DDCR, U10 INA226, U2 USBLC6-2SC6, U9A1 AP2112K-3.3, U9B1 AP2112K-3.3

Commit message: Sensor Sheet Updated
Connections:
- net +3.3V renamed +3V3
- net +3.3V_SENSOR renamed +3V3_SENSOR

Commit message: Updated and complete Schematic
Connections:
- net U10_VCC is gone; now on net +3V3_SENSOR: C7.1
- net VIN is gone; now on an unnamed net: U1.5 (EN)
Changed lines of the file:
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@@
+	)
+	(junction
+		(at 86.36 128.27)
+		(diameter 0)
+		(color 0 0 0 0)
 	)
 	(junction
@@
 	(wire
 		(pts
+			(xy 86.36 133.35) (xy 91.44 133.35)
+		)
+		(stroke
+			(width 0)
+			(type default)
+		)
+	)
+	(wire
+		(pts
 			(xy 45.72 153.67) (xy 48.26 153.67)
 		)
@@
 	(wire
 		(pts
+			(xy 86.36 128.27) (xy 86.36 133.35)
+		)
+		(stroke
+			(width 0)
+			(type default)
+		)
+	)
+	(wire
+		(pts
 			(xy 134.62 55.88) (xy 115.57 55.88)
 		)
@@
 	(wire
 		(pts
-			(xy 199.39 50.8) (xy 201.93 50.8)
+			(xy 199.39 50.8) (xy 204.47 50.8)
 		)
 		(stroke
@@
 		)
 	)
-	(hierarchical_label "VIN"
-		(shape output)
-		(at 91.44 133.35 180)
-		(effects
-			(font
-				(size 1.27 1.27)
-			)
-			(justify right)
-		)
-	)
 	(hierarchical_label "+3V3"
 		(shape output)
@@
 		)
 	)
+	(hierarchical_label "+3V3_SENSOR"
+		(shape output)
+		(at 204.47 50.8 0)
+		(effects
+			(font
+				(size 1.27 1.27)
+			)
+			(justify left)
+		)
+	)
 	(hierarchical_label "I2C1_SDA"
 		(shape bidirectional)
@@
 		)
 	)
-	(hierarchical_label "U10_VCC"
-		(shape output)
-		(at 201.93 50.8 0)
-		(effects
-			(font
-				(size 1.27 1.27)
-			)
-			(justify left)
-		)
-	)

Commit message: update
Connections:
- net USB_FS_DM renamed USB_DM
- net USB_FS_DP renamed USB_DP
Changed lines of the file:
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@@
 		)
 	)
-	(hierarchical_label "USB_FS_DP"
+	(hierarchical_label "USB_DP"
 		(shape bidirectional)
 		(at 238.76 124.46 0)
@@
 		)
 	)
-	(hierarchical_label "USB_FS_DM"
+	(hierarchical_label "USB_DM"
 		(shape bidirectional)
 		(at 245.11 137.16 0)

Commit message: Update
Parts:
- removed R26: 20mohm, Resistor_SMD:R_2512_6332Metric, symbol Device:R_Shunt
- added R26: 20m ohm, Resistor_SMD:R_2512_6332Metric, symbol Device:R
- D1: footprint SMBJ12A:DIOM4336X265N -> Library:DIOM4336X265N
- D2: footprint B0530W:DIO_B0530W -> Library:DIO_B0530W
- J1: footprint XT30PW-M:AMASS_XT30PW-M -> Library:XT30PW-M
- U1: footprint TPS563201DDCR:SOT95P280X110-6N -> Library:SOT95P280X110-6N
- U2: footprint USBLC6-2SC6:SOT95P280X145-6N -> Library:SOT95P280X145-6N
- U9B1: footprint Footprints:SOT95P285X145-5N -> Library:SOT95P285X145-5N
Connections:
- net at C1.1, C2.2, U1.3 (VIN)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: now also R26.2
- net at D1.A, F1.2, U10.10 (Vin+): now also R26.1

Commit message: updated
Parts:
- added C34: 100nF, Capacitor_SMD:C_0603_1608Metric, symbol Device:C
Connections:
- net +5V: now also U2.5, C34.1
- net GND: now also C34.2; no longer J2.A7 (D-), J2.B7 (D-), R4.1, U2.3, U2.4, U2.5
- new net: R4.1, U2.4
- new net: J2.A7 (D-), J2.B7 (D-), U2.3
Other:
- moved on the sheet: R4

Commit message: Edge Cut Made
Parts:
- U2: PACKAGE SOT-23-6 STMicroelectronics -> (none); PRICE None -> (none); PURCHASE-URL https://pricing.snapeda.com/search/part/USBLC6-2SC6/?ref=eda -> (none)
Changed lines of the file:
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@@
 			)
 		)
-		(property "PURCHASE-URL" "https://pricing.snapeda.com/search/part/USBLC6-2SC6/?ref=eda"
+		(property "Purchase-URL" "https://pricing.snapeda.com/search/part/USBLC6-2SC6/?ref=eda"
 			(at 207.01 137.16 0)
 			(hide yes)
@@
 			)
 		)
-		(property "PACKAGE" "SOT-23-6 STMicroelectronics"
+		(property "Package" "SOT-23-6 STMicroelectronics"
 			(at 207.01 137.16 0)
 			(hide yes)
@@
 			)
 		)
-		(property "PRICE" "None"
+		(property "Price" "None"
 			(at 207.01 137.16 0)
 			(hide yes)
