File: KiCAD/AERIS-H743-PCB/AERIS-H743-PCB.kicad_pcb (KiCad board)
At the start: 2 copper layers, 64 parts, among them J2 USB_C_Receptacle_USB2.0_16P, J3 Conn_01x06, Q1 Q_PMOS_GSD, SW1 SW_Push, SW2 SW_Push, U10 INA226, U3 STM32H743VITx, U5 W25Q128JVS, U9 AMS1117-3.3, U9A1 AP2112K-3.3, U9B1 AP2112K-3.3, Y1 25 MHz, Y2 32.768kHz

Commit message: update
Parts:
- added BT1: Battery, Battery:BatteryHolder_Keystone_1058_1x2032, F.Cu at (225.1, 88.7)
- added C19: 100nF, Capacitor_SMD:C_0603_1608Metric, F.Cu at (210.2, 104.2)
- added C27: 100nF, Capacitor_SMD:C_0603_1608Metric, F.Cu at (244.1, 77.6)
- added C28: 100nF, Capacitor_SMD:C_0603_1608Metric, F.Cu at (244.1, 80.1)
- added C29: 100nF, Capacitor_SMD:C_0603_1608Metric, F.Cu at (244.1, 82.6)
- added C30: 100nF, Capacitor_SMD:C_0603_1608Metric, F.Cu at (244.1, 85.1)
- added R17: 10k, Resistor_SMD:R_0603_1608Metric, F.Cu at (244.1, 87.6)
- added R18: 4.7k, Resistor_SMD:R_0603_1608Metric, F.Cu at (244.1, 90.1)
- added R19: 4.7k, Resistor_SMD:R_0603_1608Metric, F.Cu at (244.1, 92.7)
- added U4: ICM-42688-P, Package_LGA:LGA-14_3x2.5mm_P0.5mm_LayoutBorder3x4y, F.Cu at (159.6, 98.3)
- added U6: BME280, Package_LGA:Bosch_LGA-8_2.5x2.5mm_P0.65mm_ClockwisePinNumbering, F.Cu at (149.2, 95.0)
- added U7: DS3231MZ, Package_SO:SOIC-8_3.9x4.9mm_P1.27mm, F.Cu at (151.1, 89.5)
Connections:
- net /MCU_Core/+3.3V renamed /MCU_Core/+3V3
- net /POWER SECTION/+3.3V_SENSOR renamed /POWER SECTION/+3V3_SENSOR
- U10 pad 4: /POWER SECTION/I2C1_SDA -> /MCU_Core/I2C1_SDA
- U10 pad 5: /POWER SECTION/I2C1_SCL -> /MCU_Core/I2C1_SCL
- U3 pad 28: unconnected-(U3-PA4-Pad28) -> /MCU_Core/SPI1_NSS
- U3 pad 29: unconnected-(U3-PA5-Pad29) -> /MCU_Core/SPI1_SCK
- U3 pad 30: unconnected-(U3-PA6-Pad30) -> /MCU_Core/SPI1_MISO
- U3 pad 31: unconnected-(U3-PA7-Pad31) -> /MCU_Core/SPI1_MOSI
- U3 pad 95: unconnected-(U3-PB8-Pad95) -> /MCU_Core/I2C1_SCL
- U3 pad 96: unconnected-(U3-PB9-Pad96) -> /MCU_Core/I2C1_SDA

Commit message: Updated and complete Schematic
Parts:
- added C31: 100nF, Capacitor_SMD:C_0603_1608Metric, F.Cu at (163.4, 106.2)
- added C32: 100nF, Capacitor_SMD:C_0603_1608Metric, F.Cu at (163.4, 108.7)
- added C33: 100nF, Capacitor_SMD:C_0603_1608Metric, F.Cu at (132.3, 115.2)
- added D3: LED3, LED_SMD:LED_0603_1608Metric, F.Cu at (140.4, 115.2)
- added D4: LED2, LED_SMD:LED_0603_1608Metric, F.Cu at (140.4, 117.8)
- added D5: LED1, LED_SMD:LED_0603_1608Metric, F.Cu at (140.4, 120.4)
- added J10: ESC1, Connector_PinHeader_2.54mm:PinHeader_1x03_P2.54mm_Vertical, F.Cu at (132.6, 106.6)
- added J11: ESC2, Connector_PinHeader_2.54mm:PinHeader_1x03_P2.54mm_Vertical, F.Cu at (137.2, 106.6)
- added J12: ESC3, Connector_PinHeader_2.54mm:PinHeader_1x03_P2.54mm_Vertical, F.Cu at (141.8, 106.6)
- added J13: ESC4, Connector_PinHeader_2.54mm:PinHeader_1x03_P2.54mm_Vertical, F.Cu at (146.4, 106.6)
- added J5: Conn_01x02_Pin, Connector_PinHeader_2.54mm:PinHeader_1x02_P2.54mm_Vertical, F.Cu at (163.7, 117.2)
- added J6: Conn_01x02_Pin, Connector_PinHeader_2.54mm:PinHeader_1x02_P2.54mm_Vertical, F.Cu at (168.3, 117.2)
- added J7: Conn_01x04_Pin, Connector_PinHeader_2.54mm:PinHeader_1x04_P2.54mm_Vertical, F.Cu at (159.1, 107.2)
- added R20: 120 ohm DNP, Resistor_SMD:R_0603_1608Metric, F.Cu at (163.4, 111.2)
- added R21: 120 ohm DNP, Resistor_SMD:R_0603_1608Metric, F.Cu at (163.4, 113.7)
- added R22: 330 ohm, Resistor_SMD:R_0603_1608Metric, F.Cu at (132.3, 117.7)
- added R23: 10 Kohm (pulldown), Resistor_SMD:R_0603_1608Metric, F.Cu at (132.3, 120.2)
- added R24: 10Kohm (PullDown), Resistor_SMD:R_0603_1608Metric, F.Cu at (132.3, 122.7)
- added R25: 330 ohm, Resistor_SMD:R_0603_1608Metric, F.Cu at (132.3, 125.2)
- added R27: 10kohm(PD), Resistor_SMD:R_0603_1608Metric, F.Cu at (132.3, 127.8)
- added R28: 220ohm, Resistor_SMD:R_0603_1608Metric, F.Cu at (136.3, 115.2)
- added R29: 10kohm(PD), Resistor_SMD:R_0603_1608Metric, F.Cu at (136.3, 117.7)
- added R30: 330 ohm, Resistor_SMD:R_0603_1608Metric, F.Cu at (136.3, 120.2)
- added R31: 10Kohm(PU), Resistor_SMD:R_0603_1608Metric, F.Cu at (136.3, 122.7)
- added R32: 330 ohm, Resistor_SMD:R_0603_1608Metric, F.Cu at (136.3, 125.2)
- added SW3: SW_Push, Button_Switch_SMD:SW_SPST_B3U-1000P, F.Cu at (145.3, 116.1)
- added U11: MAX3485, Package_SO:SOIC-8_3.9x4.9mm_P1.27mm, F.Cu at (214.2, 117.0)
- added U8: SN65HVD230, Package_SO:SOIC-8_3.9x4.9mm_P1.27mm, F.Cu at (214.2, 110.4)
- moved R17 57.7 mm to (195.6, 118.7)
- moved C29 51.8 mm to (193.2, 92.1)
- moved R19 50.0 mm to (200.7, 117.5)
- moved R18 49.4 mm to (200.7, 113.7)
- moved C28 47.4 mm to (199.4, 95.9)
- moved C27 43.3 mm to (206.9, 99.7)
- moved BT1 42.7 mm to (186.5, 106.7)
- moved C30 37.1 mm to (207.8, 92.7)
Connections:
- net /MCU_Core/+3V3 renamed /COMMUNICATION/+3V3

Commit message: Update
Parts:
- added D1: SMBJ12A, Library:DIOM4336X265N, F.Cu at (235.3, 66.8)
- added D2: B0530W, Library:DIO_B0530W, F.Cu at (234.1, 70.9)
- added D6: LED_RGB, LED_SMD:LED_RGB_5050-6, F.Cu at (214.0, 66.4)
- added J1: XT30PW-M, Library:XT30PW-M, F.Cu at (219.8, 76.4)
- added J4: 1040310811, Library:104031-0811_MOL, F.Cu at (252.7, 95.5)
- added R26: 20m ohm, Resistor_SMD:R_2512_6332Metric, F.Cu at (135.3, 91.5)
- added U1: TPS563201DDCR, Library:SOT95P280X110-6N, F.Cu at (240.0, 71.6)
- added U2: USBLC6-2SC6, Library:SOT95P280X145-6N, F.Cu at (233.9, 74.7)
- added Y2: 32.768KHz, Crystal:Crystal_SMD_3215-2Pin_3.2x1.5mm, F.Cu at (220.5, 100.9)
- U9B1: footprint Footprints:SOT95P285X145-5N -> Library:SOT95P285X145-5N
Connections:
- net /MCU_Core/I2C1_SCL renamed /I2C1_SCL
- net /MCU_Core/I2C1_SDA renamed /I2C1_SDA
- C19 pad 2: /COMMUNICATION/+3V3 -> /3.3
- C21 pad 1: /COMMUNICATION/+3V3 -> /3.3
- C22 pad 1: /COMMUNICATION/+3V3 -> /3.3
- C23 pad 1: /COMMUNICATION/+3V3 -> /3.3
- C24 pad 1: /COMMUNICATION/+3V3 -> /3.3
- C25 pad 1: /COMMUNICATION/+3V3 -> /3.3
- C26 pad 1: /COMMUNICATION/+3V3 -> /3.3
- C27 pad 2: /POWER SECTION/+3V3_SENSOR -> /3.3_Sensor
- C28 pad 1: /POWER SECTION/+3V3_SENSOR -> /3.3_Sensor
- C29 pad 1: /POWER SECTION/+3V3_SENSOR -> /3.3_Sensor
- C31 pad 2: /COMMUNICATION/+3V3 -> /3.3
- C32 pad 2: /COMMUNICATION/+3V3 -> /3.3
- C33 pad 1: unconnected-(C33-Pad1) -> /U_BTN
- C33 pad 2: unconnected-(C33-Pad2) -> GND
- C5 pad 1: /COMMUNICATION/+3V3 -> /3.3
- C5b1 pad 1: /COMMUNICATION/+3V3 -> /3.3
- C5d1 pad 1: /POWER SECTION/+3V3_SENSOR -> /3.3_Sensor
- C7 pad 1: /POWER SECTION/U10_VCC -> /3.3_Sensor
- C9 pad 1: /COMMUNICATION/+3V3 -> /3.3
- D4 pad 1: unconnected-(D4-K-Pad1) -> GND
- D4 pad 2: unconnected-(D4-A-Pad2) -> Net-(D4-A)
- D5 pad 1: unconnected-(D5-K-Pad1) -> GND
- D5 pad 2: unconnected-(D5-A-Pad2) -> Net-(D5-A)
- FB1 pad 2: /COMMUNICATION/+3V3 -> /3.3
- J10 pad 1: /Connectors and Indicators/PE9 -> /PE9
- J11 pad 1: /Connectors and Indicators/PE11 -> /PE11
- J12 pad 1: /Connectors and Indicators/PE13 -> /PE13
- J13 pad 1: /Connectors and Indicators/PE14 -> /PE14
- J3 pad 1: /COMMUNICATION/+3V3 -> /3.3
- J7 pad 1: /COMMUNICATION/GPS_TX(PE1) -> /GPS_TX
- J7 pad 2: /COMMUNICATION/GPS_RX(PE0) -> /GPS_RX
- J7 pad 3: /COMMUNICATION/+3V3 -> /3.3
- R10 pad 1: /COMMUNICATION/+3V3 -> /3.3
- R10 pad 2: /Memory and Storage/QSPI_IO2 -> /QSPI_IO2
- R11 pad 1: /COMMUNICATION/+3V3 -> /3.3
- R11 pad 2: /Memory and Storage/QSPI_IO3 -> /QSPI_IO3
- R12 pad 1: /COMMUNICATION/+3V3 -> /3.3
- R12 pad 2: /Memory and Storage/SDMMC_CMD -> /SDMMC_CMD
- R13 pad 1: /COMMUNICATION/+3V3 -> /3.3
- R13 pad 2: /Memory and Storage/SDMMC_D0 -> /SDMMC_D0
- R14 pad 1: /COMMUNICATION/+3V3 -> /3.3
- R14 pad 2: /Memory and Storage/SDMMC_D1 -> /SDMMC_D1
- R15 pad 1: /COMMUNICATION/+3V3 -> /3.3
- R15 pad 2: /Memory and Storage/SDMMC_D2 -> /SDMMC_D2
- R16 pad 1: /COMMUNICATION/+3V3 -> /3.3
- R16 pad 2: /Memory and Storage/SDMMC_D3 -> /SDMMC_D3
- R17 pad 2: /POWER SECTION/+3V3_SENSOR -> /3.3_Sensor
- R18 pad 2: /POWER SECTION/+3V3_SENSOR -> /3.3_Sensor
- R19 pad 2: /POWER SECTION/+3V3_SENSOR -> /3.3_Sensor
- R22 pad 1: unconnected-(R22-Pad1) -> /3.3
- R22 pad 2: unconnected-(R22-Pad2) -> Net-(D5-A)
- R23 pad 2: /Connectors and Indicators/PE11 -> /PE11
- R24 pad 2: /Connectors and Indicators/PE9 -> /PE9
- R25 pad 1: unconnected-(R25-Pad1) -> Net-(D4-A)
- R25 pad 2: unconnected-(R25-Pad2) -> /S_LED
- R27 pad 2: /Connectors and Indicators/PE13 -> /PE13
- R28 pad 1: unconnected-(R28-Pad1) -> Net-(D6-RA)
- R28 pad 2: unconnected-(R28-Pad2) -> /RGB_R
- R29 pad 2: /Connectors and Indicators/PE14 -> /PE14
- R30 pad 1: unconnected-(R30-Pad1) -> Net-(D6-BA)
- R30 pad 2: unconnected-(R30-Pad2) -> /RGB_B
- R31 pad 1: unconnected-(R31-Pad1) -> /3.3
- R31 pad 2: unconnected-(R31-Pad2) -> /U_BTN
- R32 pad 1: unconnected-(R32-Pad1) -> /RGB_G
- R32 pad 2: unconnected-(R32-Pad2) -> Net-(D6-GA)
- R4 pad 2: /POWER SECTION/USB_FS_DM -> /USB_DM
- R5 pad 2: /POWER SECTION/USB_FS_DP -> /USB_DP
- SW2 pad 2: /COMMUNICATION/+3V3 -> /3.3
- SW3 pad 1: unconnected-(SW3-Pad1) -> /U_BTN
- SW3 pad 2: unconnected-(SW3-Pad2) -> GND
- U10 pad 6: /POWER SECTION/+3V3_SENSOR -> /3.3_Sensor
- U11 pad 1: /COMMUNICATION/RS485_RX -> /RS485_RX
- U11 pad 2: /COMMUNICATION/RS485_DE -> /RS485_DE
- U11 pad 3: /COMMUNICATION/RS485_DE -> /RS485_DE
- U11 pad 4: /COMMUNICATION/RS485_TX -> /RS485_TX
- U11 pad 8: /COMMUNICATION/+3V3 -> /3.3
- U3 pad 1: unconnected-(U3-PE2-Pad1) -> /QSPI_IO2
- U3 pad 100: /COMMUNICATION/+3V3 -> /3.3
- U3 pad 11: /COMMUNICATION/+3V3 -> /3.3
- U3 pad 15: unconnected-(U3-PC0-Pad15) -> /IMU_INT1
- U3 pad 16: unconnected-(U3-PC1-Pad16) -> /U_BTN
- U3 pad 17: unconnected-(U3-PC2_C-Pad17) -> /S_LED
- U3 pad 18: unconnected-(U3-PC3_C-Pad18) -> /RGB_R
- U3 pad 27: /COMMUNICATION/+3V3 -> /3.3
- U3 pad 32: unconnected-(U3-PC4-Pad32) -> /RGB_G
- U3 pad 33: unconnected-(U3-PC5-Pad33) -> /RGB_B
- U3 pad 36: unconnected-(U3-PB2-Pad36) -> /QSPI_CLK
- U3 pad 39: unconnected-(U3-PE9-Pad39) -> /PE9
- U3 pad 41: unconnected-(U3-PE11-Pad41) -> /PE11
- U3 pad 43: unconnected-(U3-PE13-Pad43) -> /PE13
- U3 pad 44: unconnected-(U3-PE14-Pad44) -> /PE14
- U3 pad 50: /COMMUNICATION/+3V3 -> /3.3
- U3 pad 55: unconnected-(U3-PD8-Pad55) -> /RS485_TX
- U3 pad 56: unconnected-(U3-PD9-Pad56) -> /RS485_RX
- U3 pad 57: unconnected-(U3-PD10-Pad57) -> /RS485_DE
- U3 pad 58: unconnected-(U3-PD11-Pad58) -> /QSPI_IO0
- U3 pad 59: unconnected-(U3-PD12-Pad59) -> /QSPI_IO1
- U3 pad 60: unconnected-(U3-PD13-Pad60) -> /QSPI_IO3
- U3 pad 65: unconnected-(U3-PC8-Pad65) -> /SDMMC_D0
- U3 pad 66: unconnected-(U3-PC9-Pad66) -> /SDMMC_D1
- U3 pad 70: unconnected-(U3-PA11-Pad70) -> /USB_DM
- U3 pad 71: unconnected-(U3-PA12-Pad71) -> /USB_DP
- U3 pad 75: /COMMUNICATION/+3V3 -> /3.3
- U3 pad 78: unconnected-(U3-PC10-Pad78) -> /SDMMC_D2
- U3 pad 79: unconnected-(U3-PC11-Pad79) -> /SDMMC_D3
- U3 pad 80: unconnected-(U3-PC12-Pad80) -> /SDMMC_CLK
- U3 pad 81: unconnected-(U3-PD0-Pad81) -> /F_RX
- U3 pad 82: unconnected-(U3-PD1-Pad82) -> /F_TX
- U3 pad 83: unconnected-(U3-PD2-Pad83) -> /SDMMC_CMD
- U3 pad 92: unconnected-(U3-PB6-Pad92) -> /QSPI_NCS
- U3 pad 97: unconnected-(U3-PE0-Pad97) -> /GPS_RX
- U3 pad 98: unconnected-(U3-PE1-Pad98) -> /GPS_TX
- U4 pad 4: /SENSORS/IMU_INT1 -> /IMU_INT1
- U4 pad 5: /POWER SECTION/+3V3_SENSOR -> /3.3_Sensor
- U4 pad 8: /POWER SECTION/+3V3_SENSOR -> /3.3_Sensor
- U5 pad 1: /Memory and Storage/QSPI_NCS -> /QSPI_NCS
- U5 pad 2: /Memory and Storage/QSPI_IO1 -> /QSPI_IO1
- U5 pad 3: /Memory and Storage/QSPI_IO2 -> /QSPI_IO2
- U5 pad 5: /Memory and Storage/QSPI_IO0 -> /QSPI_IO0
- U5 pad 6: /Memory and Storage/QSPI_CLK -> /QSPI_CLK
- U5 pad 7: /Memory and Storage/QSPI_IO3 -> /QSPI_IO3
- U5 pad 8: /COMMUNICATION/+3V3 -> /3.3
- U6 pad 2: /POWER SECTION/+3V3_SENSOR -> /3.3_Sensor
- U6 pad 6: /POWER SECTION/+3V3_SENSOR -> /3.3_Sensor
- U6 pad 8: /POWER SECTION/+3V3_SENSOR -> /3.3_Sensor
- U7 pad 2: /POWER SECTION/+3V3_SENSOR -> /3.3_Sensor
- U8 pad 1: /COMMUNICATION/FDCAN1_TX -> /F_TX
- U8 pad 3: /COMMUNICATION/+3V3 -> /3.3
- U8 pad 4: /COMMUNICATION/FDCAN1_RX -> /F_RX
- U9A1 pad 5: /COMMUNICATION/+3V3 -> /3.3
- U9B1 pad 5: /POWER SECTION/+3V3_SENSOR -> /3.3_Sensor

Commit message: updated
Parts:
- added C34: 100nF, Capacitor_SMD:C_0603_1608Metric, F.Cu at (213.6, 49.0)
- added J1: XT30PW-M, Library:XT30PW-M, F.Cu at (255.8, 67.4)
- added J1: XT30PW-M, Connector_AMASS:AMASS_XT30PW-M_1x02_P2.50mm_Horizontal, F.Cu at (9.68, 13.6)
- added U1: TPS563201DDCR, Library:SOT95P280X110-6N, F.Cu at (239.5, 55.7)
- added U2: USBLC6-2SC6, Library:SOT95P280X145-6N, F.Cu at (222.5, 45.6)
Connections:
- J2 pad A7: GND -> Net-(J2-D--PadA7)
- J2 pad B7: GND -> Net-(J2-D--PadA7)
- R4 pad 1: GND -> Net-(R4-Pad1)
- U4 pad 9: GND -> unconnected-(U4-INT2/FSYNC/CLKIN-Pad9)
- U6 pad 5: GND -> unconnected-(U6-SDO-Pad5)

Commit message: Edge Cut Made
Parts:
- removed the J1 at (9.68, 13.6)
- moved C10 215.4 mm to (-41.7, 23.3)
- moved C12 215.4 mm to (-37.7, 15.8)
- moved C15 215.4 mm to (-37.7, 23.3)
- moved C19 215.4 mm to (4.41, 40.4)
- moved C2 215.4 mm to (-71.3, 0.55)
- moved C28 215.4 mm to (-6.36, 32.1)
- moved C31 215.4 mm to (-42.4, 42.4)
- moved C33 215.4 mm to (-73.4, 51.4)
- moved C5 215.4 mm to (-41.7, 15.8)
- moved C5a1 215.4 mm to (-71.3, 9.58)
- moved C5c1 215.4 mm to (-15.7, 2.11)
- moved J4 215.4 mm to (47.0, 31.8)
- moved J6 215.4 mm to (-37.5, 53.5)
- moved Q1 215.4 mm to (-62.6, 17.8)
- moved R18 215.4 mm to (-5.09, 49.9)
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Other:
- board outline added: 141.4 x 141.4 mm

Commit message: PCB Design process 20% complete
Parts:
- removed the J1 at (50.1, 3.57)
- removed the J1 at (14.0, 12.6)
- removed the U1 at (34.2, 7.80)
- added J1: XT30PW-M, Library:XT30PW-M, B.Cu at (153.0, 109.9)
- C1, C2, C3, C4, C5a1, C5b1, C5c1, C5d1, D1, F1, J4, L1, Q1, R1, R2, R26, R3, U1, U10, U9A1, U9B1: moved to B.Cu
- moved C5b1 257.4 mm to (170.2, 101.6), turned to -90 degrees
- moved C5a1 256.1 mm to (167.6, 101.6), turned to -90 degrees
- moved R1 244.9 mm to (156.8, 96.5), turned to 180 degrees
- moved J11 243.5 mm to (173.2, 71.6), turned to -135 degrees
- moved J13 240.4 mm to (170.9, 111.7), turned to 135 degrees
- moved C2 239.9 mm to (144.1, 106.0), turned to 90 degrees
- moved C1 239.0 mm to (141.6, 106.0), turned to -90 degrees
- moved R26 238.4 mm to (158.8, 93.3), turned to 180 degrees
- moved J2 237.2 mm to (150.1, 103.3)
- moved C3 234.0 mm to (139.1, 106.0), turned to -90 degrees
- moved R3 231.8 mm to (143.5, 99.1), turned to 180 degrees
- moved C4 231.1 mm to (139.1, 102.2), turned to 90 degrees
- moved R2 229.4 mm to (139.7, 99.1), turned to 180 degrees
- moved Q1 229.1 mm to (153.0, 95.2), turned to 90 degrees
- moved L1 222.7 mm to (141.6, 110.5)
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Other:
- outline, holes or cut-outs redrawn
- copper layers 2 -> 6
- board text added: "ESC1"
- board text added: "ESC2"
- board text added: "ESC3"
- board text added: "ESC4"

Commit message: Component Placement Done
Parts:
- removed D3: LED3, LED_SMD:LED_0603_1608Metric
- BT1, C25, C26, C27, C28, C29, C30, D1, R18, R19, R26, U6, U7: moved to B.Cu
- moved D2 250.2 mm to (177.8, 104.1), turned to 135 degrees
- moved R4 249.5 mm to (163.4, 100.3)
- moved R5 249.5 mm to (163.4, 102.8)
- moved U9 246.4 mm to (170.2, 99.1)
- moved R28 233.0 mm to (160.0, 92.1)
- moved R30 232.8 mm to (160.0, 95.9)
- moved R32 231.7 mm to (160.0, 94.0)
- moved R6 231.4 mm to (138.4, 116.2), turned to 45 degrees
- moved R7 231.4 mm to (140.9, 113.7), turned to 45 degrees
- moved C5 228.7 mm to (141.3, 86.4)
- moved C7 226.3 mm to (141.2, 93.3)
- moved R22 224.4 mm to (144.3, 108.0)
- moved R23 223.0 mm to (144.1, 105.4)
- moved R25 222.9 mm to (144.0, 110.5)
- moved R29 218.9 mm to (144.0, 102.9)
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Other:
- outline, holes or cut-outs redrawn

Commit message: working Routing
Parts:
- moved D1 12.5 mm to (123.2, 69.8)
Routing:
- net Net-(BT1-+): track 0.00 -> 83.2 mm
- net /SDMMC_D3: track 0.00 -> 63.7 mm, vias 0 -> 2
- net Net-(U10-Vin+): track 0.00 -> 60.8 mm
- net /I2C1_SCL: track 0.00 -> 60.7 mm, vias 0 -> 3
- net /I2C1_SDA: track 0.00 -> 58.7 mm, vias 0 -> 3
- net /SDMMC_CLK: track 0.00 -> 52.3 mm, vias 0 -> 1
- net /PE9: track 0.00 -> 51.0 mm, vias 0 -> 1
- net Net-(U1-EN): track 0.00 -> 38.6 mm
- net /SDMMC_CMD: track 0.00 -> 38.4 mm, vias 0 -> 1
- net Net-(J3-Pin_4): track 0.00 -> 38.3 mm, vias 0 -> 1
- net /MCU_Core/VSSA: track 0.00 -> 37.5 mm, vias 0 -> 6
- net Net-(J3-Pin_6): track 0.00 -> 36.8 mm, vias 0 -> 1
- net Net-(J3-Pin_2): track 0.00 -> 35.9 mm, vias 0 -> 1
- net /PE13: track 0.00 -> 35.0 mm, vias 0 -> 1
- net /SDMMC_D2: track 0.00 -> 33.7 mm, vias 0 -> 1
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- added copper zone on In2.Cu, net /3.3
