File: KiCAD/AERIS-H743-PCB/AERIS-H743-PCB.kicad_pcb (KiCad board)
At the start: 6 copper layers, 141.4 x 141.4 mm, 114 parts, among them J1 XT30PW-M, J10 ESC1, J11 ESC2, J12 ESC3, J13 ESC4, J2 USB_C_Receptacle_USB2.0_16P, J3 Conn_01x06, J4 1040310811, J5 Conn_01x02_Pin, J6 Conn_01x02_Pin, J7 Conn_01x04_Pin, Q1 Q_PMOS_GSD, SW1 SW_Push, SW2 SW_Push, SW3 SW_Push, U1 TPS563201DDCR, U10 INA226, U11 MAX3485, U2 USBLC6-2SC6, U3 STM32H743VITx, U4 ICM-42688-P, U5 W25Q128JVS, U6 BME280, U7 DS3231MZ, U8 SN65HVD230, U9 AMS1117-3.3, U9A1 AP2112K-3.3, U9B1 AP2112K-3.3, Y1 25 MHz, Y2 32.768KHz, Y2 32.768kHz

Commit message: Completed
Routing:
- net GND: track 0.00 -> 272.5 mm, vias 0 -> 30
- net /MCU_Core/NRST: track 0.00 -> 77.0 mm, vias 0 -> 4
- net /QSPI_IO2: track 0.00 -> 67.7 mm, vias 0 -> 4
- net /3.3: track 6.30 -> 71.1 mm, vias 2 -> 20
- net /POWER SECTION/GND: track 0.00 -> 64.0 mm, vias 0 -> 2
- net /MCU_Core/PH1: track 0.00 -> 62.6 mm, vias 0 -> 2
- net /MCU_Core/SPI1_NSS: track 0.00 -> 55.8 mm
- net /MCU_Core/PC15: track 0.00 -> 50.6 mm, vias 0 -> 3
- net /F_RX: track 0.00 -> 47.2 mm, vias 0 -> 2
- net /F_TX: track 0.00 -> 41.7 mm, vias 0 -> 2
- net /QSPI_IO3: track 0.00 -> 40.3 mm, vias 0 -> 3
- net /USB_DP: track 0.00 -> 38.3 mm, vias 0 -> 2
- net /PE14: track 33.3 -> 70.0 mm, vias 1 -> 3
- net /S_LED: track 0.00 -> 36.7 mm, vias 0 -> 2
- net Net-(C12-Pad1): track 0.00 -> 35.8 mm, vias 0 -> 2
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- added copper zone on In1.Cu, net /3.3
- added copper zone on In3.Cu, net /3.3_Sensor
- added copper zone on In2.Cu, net GND
- removed copper zone on In2.Cu, net /3.3
